File: 0.2/compact/ferris.kicad_pcb (KiCad board)
At the start: 2 copper layers, 208.8 x 86.8 mm, 109 parts, among them J1 TYPE-C-31-M-12, K0_0 KEYSW, K0_1 KEYSW, K0_2 KEYSW, K0_3 KEYSW, K0_4 KEYSW, K0_5 KEYSW, K0_6 KEYSW, K0_7 KEYSW, K0_8 KEYSW, K0_9 KEYSW, K1_0 KEYSW, K1_1 KEYSW, K1_2 KEYSW, K1_3 KEYSW, K1_4 KEYSW, K1_5 KEYSW, K1_6 KEYSW, K1_7 KEYSW, K1_8 KEYSW, K1_9 KEYSW, K2_0 KEYSW, K2_1 KEYSW, K2_2 KEYSW, K2_3 KEYSW, K2_4 KEYSW, K2_5 KEYSW, K2_6 KEYSW, K2_7 KEYSW, K2_8 KEYSW, K2_9 KEYSW, K3_3 KEYSW, K3_4 KEYSW, K3_5 KEYSW, K3_6 KEYSW, Q1 PDTC123JT,215, SW1 B3U-1000P, U1 STM32F072CBT6, U2 MCP23017-E/SO, U3 MCP1700T-3302E/TT, U4 SRV05-4

Commit message: split pcb and 3d casing
Parts:
- removed the G*** at (117.1, 34.8)
- removed mouse-bite-2mm-slot (x3): VAL**, panelization:mouse-bite-2mm-slot-with-space-for-track
- moved C12 9.84 mm to (139.8, 72.1)
- moved C13 9.84 mm to (131.8, 72.1)
- moved D0_5 9.84 mm to (151.8, 25.9)
- moved D0_6 9.84 mm to (169.8, 23.4)
- moved D0_7 9.84 mm to (187.8, 17.9)
- moved D0_8 9.84 mm to (205.8, 24.9)
- moved D0_9 9.84 mm to (223.8, 36.8)
- moved D1_5 9.84 mm to (151.8, 42.9)
- moved D1_6 9.84 mm to (169.8, 40.4)
- moved D1_7 9.84 mm to (187.8, 34.9)
- moved D1_8 9.84 mm to (205.8, 41.8)
- moved D1_9 9.84 mm to (223.8, 53.9)
- moved D2_5 9.84 mm to (151.8, 59.9)
- moved D2_6 9.84 mm to (169.8, 57.3)
- moved D2_7 9.84 mm to (187.8, 51.9)
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Routing:
- net GND: track 214.9 -> 183.9 mm, vias 23 -> 22
Other:
- board size 208.8 x 86.8 mm -> 218.6 x 87.3 mm
- net class Default removed
- net class Power removed
- board text removed: "Ferris Compact - v0.2.1 by @pierrec83 Minimalism shall prevail :D * Split, 34 Keys * Kailh Choc footprints: pg1350 * Choc spacing: 17x18mm * Microcontroller: STM32FO72 * IO Expander: MCP23017 * USB C * All MCU pins are broken out * Nothing frivolous Fully open source design: github.com/pierrechevalier83/ferris"
